File: Bare_ESP32.brd (EAGLE design)
At the start: 21.3 x 22.8 mm, 18 parts, among them U1 ESP32-PICO-D4

Commit message: Add files via upload
Parts:
- added C1: 1pF, SparkFun-Capacitors:0402
- added L2.7: 2.7nH, L-07C2N7SV6T:INDC1005X60N
- added L3.9: 3.9nH, L-07C2N7SV6T:INDC1005X60N
- moved ANT 43.3 mm to (17.8, 2.54), turned to 270 degrees
- moved BOOT/IO0 35.8 mm to (3.81, 19.1)
- moved C5 35.8 mm to (14.0, 16.5)
- moved C7 35.8 mm to (3.81, 16.5)
- moved D2 35.8 mm to (1.91, 9.53)
- moved GND 35.8 mm to (5.08, 2.54)
- moved R1 35.8 mm to (14.0, 12.7)
- moved R2 35.8 mm to (3.81, 10.2)
- moved R3 35.8 mm to (11.4, 2.54)
- moved R4 35.8 mm to (8.89, 16.5)
- moved RESET/EN 35.8 mm to (14.0, 19.1)
- moved RX 35.8 mm to (5.08, 5.08)
- moved TX 35.8 mm to (7.62, 5.08)
- moved U1 35.8 mm to (8.89, 11.4)
- moved VCC 35.8 mm to (7.62, 2.54)
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Connections:
- new net N$1: C1.2, L2.7.1, L3.9.1
- new net N$7: ANT.1, L3.9.2
- net GND: now also L2.7.2
- net N$4: now also C1.1; no longer ANT.1
Routing:
- net +3V3: track 92.2 -> 98.9 mm, vias 0 -> 2
- net N$1: track 0.00 -> 4.70 mm
- net GND: track 101.9 -> 104.4 mm, vias 11 -> 14
- net N$7: track 0.00 -> 1.80 mm
- net N$4: track 5.82 -> 6.73 mm
- added copper zone on layer 16, net GND
Other:
- board size 21.3 x 22.8 mm -> 21.3 x 22.9 mm
- board text added: "C1"
- board text added: "Green"
- board text added: "L2.7nH"
- board text added: "L3.9nH"
