File: Bare_ESP32.sch (EAGLE design)
At the start: 18 parts, among them U1 ESP32-PICO-D4

Commit message: Add files via upload
Parts:
- added C1: 1pF, SparkFun-Capacitors:0.1UF-0402-16V-10%
- added L2.7: 2.7nH, L-07C2N7SV6T:L-07C2N7SV6T
- added L3.9: 3.9nH, L-07C2N7SV6T:L-07C2N7SV6T
Connections:
- new net N$1: C1.2, L2.7.1, L3.9.1
- new net N$7: ANT.1, L3.9.2
- net GND: now also L2.7.2
- net N$4: now also C1.1; no longer ANT.1
Other:
- moved on the sheet: ANT
Changed lines of the file:
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@@
 <?xml version="1.0" encoding="utf-8"?>
 <!DOCTYPE eagle SYSTEM "eagle.dtd">
-<eagle version="9.4.0">
+<eagle version="9.5.2">
 <drawing>
 <settings>
@@
 <layer number="18" name="Vias" color="2" fill="1" visible="no" active="no"/>
 <layer number="19" name="Unrouted" color="6" fill="1" visible="no" active="no"/>
-<layer number="20" name="Dimension" color="15" fill="1" visible="no" active="no"/>
+<layer number="20" name="Dimension" color="24" fill="1" visible="no" active="no"/>
 <layer number="21" name="tPlace" color="7" fill="1" visible="no" active="no"/>
 <layer number="22" name="bPlace" color="7" fill="1" visible="no" active="no"/>
@@
 <part name="RX" library="testpad" library_urn="urn:adsk.eagle:library:385" deviceset="TP" device="TP14SQ" package3d_urn="urn:adsk.eagle:package:27984/1"/>
 <part name="TX" library="testpad" library_urn="urn:adsk.eagle:library:385" deviceset="TP" device="TP14SQ" package3d_urn="urn:adsk.eagle:package:27984/1"/>
-<part name="ANT" library="SMT_small_antenna" deviceset="2450AT18A100E" device=""/>
 <part name="VCC" library="testpad" library_urn="urn:adsk.eagle:library:385" deviceset="TP" device="TP14SQ" package3d_urn="urn:adsk.eagle:package:27984/1"/>
 <part name="GND" library="testpad" library_urn="urn:adsk.eagle:library:385" deviceset="TP" device="TP14SQ" package3d_urn="urn:adsk.eagle:package:27984/1"/>
@@
 <part name="+3V6" library="supply1" library_urn="urn:adsk.eagle:library:371" deviceset="+3V3" device=""/>
 <part name="ORANGE" library="BeagleBone_Blue_R3" library_urn="urn:adsk.eagle:library:5828899" deviceset="LED-ORANGE" device="0603" package3d_urn="urn:adsk.eagle:package:5829998/10"/>
+<part name="C1" library="SparkFun-Capacitors" library_urn="urn:adsk.eagle:library:510" deviceset="0.1UF" device="-0402-16V-10%" package3d_urn="urn:adsk.eagle:package:37413/1" value="1pF"/>
+<part name="L2.7" library="L-07C2N7SV6T" deviceset="L-07C2N7SV6T" device="" value="2.7nH"/>
+<part name="L3.9" library="L-07C2N7SV6T" deviceset="L-07C2N7SV6T" device="" value="3.9nH"/>
+<part name="ANT" library="SMT_small_antenna" deviceset="2450AT18A100E" device=""/>
 </parts>
 <sheets>
@@
 <attribute name="NAME" x="57.15" y="62.23" size="1.778" layer="95"/>
 </instance>
-<instance part="ANT" gate="G$1" x="93.98" y="43.18" smashed="yes">
-<attribute name="NAME" x="91.18735" y="53.3661" size="1.27523125" layer="95"/>
-<attribute name="VALUE" x="86.23908125" y="35.5625" size="1.273009375" layer="96"/>
-</instance>
 <instance part="VCC" gate="G$1" x="-22.86" y="86.36" smashed="yes">
 <attribute name="NAME" x="-24.13" y="87.63" size="1.778" layer="95"/>
@@
 <attribute name="VALUE" x="61.722" y="39.37" size="1.778" layer="96" rot="R90"/>
 </instance>
-<instance part="+3V6" gate="G$1" x="58.42" y="53.34" smashed="yes">
-<attribute name="VALUE" x="55.88" y="48.26" size="1.778" layer="96" rot="R90"/>
+<instance part="+3V6" gate="G$1" x="58.42" y="50.8" smashed="yes">
+<attribute name="VALUE" x="55.88" y="45.72" size="1.778" layer="96" rot="R90"/>
 </instance>
 <instance part="ORANGE" gate="G$1" x="66.04" y="96.52" smashed="yes" rot="R90">
 <attribute name="NAME" x="70.612" y="100.076" size="1.778" layer="95" rot="R180"/>
+</instance>
+<instance part="C1" gate="G$1" x="91.44" y="53.34" smashed="yes" rot="R90">
+<attribute name="NAME" x="88.519" y="54.864" size="1.778" layer="95" font="vector" rot="R90"/>
+<attribute name="VALUE" x="92.456" y="50.419" size="1.778" layer="96" font="vector" rot="R180"/>
+</instance>
+<instance part="L2.7" gate="G$1" x="99.06" y="53.34" smashed="yes" rot="R270">
+<attribute name="NAME" x="97.79" y="44.45" size="1.778" layer="95" rot="R270" align="center-left"/>
+</instance>
+<instance part="L3.9" gate="G$1" x="104.14" y="53.34" smashed="yes">
+<attribute name="NAME" x="110.49" y="52.07" size="1.778" layer="95" align="center-left"/>
+</instance>
+<instance part="ANT" gate="G$1" x="127" y="58.42" smashed="yes">
+<attribute name="NAME" x="124.20735" y="68.6061" size="1.27523125" layer="95"/>
 </instance>
 </instances>
@@
 <wire x1="5.08" y1="40.64" x2="5.08" y2="48.26" width="0.1524" layer="91"/>
 <junction x="5.08" y="48.26"/>
-</segment>
-</net>
-<net name="N$4" class="0">
-<segment>
-<pinref part="U1" gate="G$1" pin="LNA_IN"/>
-<wire x1="53.34" y1="53.34" x2="86.36" y2="53.34" width="0.1524" layer="91"/>
-<pinref part="ANT" gate="G$1" pin="1"/>
-<wire x1="93.98" y1="38.1" x2="86.36" y2="38.1" width="0.1524" layer="91"/>
-<wire x1="86.36" y1="38.1" x2="86.36" y2="53.34" width="0.1524" layer="91"/>
 </segment>
 </net>
@@
 <wire x1="55.88" y1="7.62" x2="55.88" y2="-2.54" width="0.1524" layer="91"/>
 <pinref part="ORANGE" gate="G$1" pin="C"/>
+<pinref part="L2.7" gate="G$1" pin="2"/>
+<wire x1="99.06" y1="33.02" x2="99.06" y2="-2.54" width="0.1524" layer="91"/>
+<wire x1="99.06" y1="-2.54" x2="76.2" y2="-2.54" width="0.1524" layer="91"/>
+<junction x="76.2" y="-2.54"/>
 </segment>
 </net>
@@
 <pinref part="R4" gate="G$1" pin="2"/>
 <pinref part="+3V6" gate="G$1" pin="+3V3"/>
-<wire x1="58.42" y1="48.26" x2="58.42" y2="50.8" width="0.1524" layer="91"/>
 </segment>
 </net>
@@
 </segment>
 </net>
+<net name="N$4" class="0">
+<segment>
+<wire x1="53.34" y1="53.34" x2="86.36" y2="53.34" width="0.1524" layer="91"/>
+<pinref part="C1" gate="G$1" pin="1"/>
+<pinref part="U1" gate="G$1" pin="LNA_IN"/>
+</segment>
+</net>
+<net name="N$7" class="0">
+<segment>
+<pinref part="L3.9" gate="G$1" pin="2"/>
+<wire x1="127" y1="53.34" x2="124.46" y2="53.34" width="0.1524" layer="91"/>
+<pinref part="ANT" gate="G$1" pin="1"/>
+</segment>
+</net>
+<net name="N$1" class="0">
+<segment>
+<pinref part="C1" gate="G$1" pin="2"/>
+<pinref part="L2.7" gate="G$1" pin="1"/>
+<wire x1="93.98" y1="53.34" x2="99.06" y2="53.34" width="0.1524" layer="91"/>
+<pinref part="L3.9" gate="G$1" pin="1"/>
+<wire x1="104.14" y1="53.34" x2="99.06" y2="53.34" width="0.1524" layer="91"/>
+<junction x="99.06" y="53.34"/>
+</segment>
+</net>
